File: Schematics/EAGLE/v9/ardustatversion9.brd (EAGLE design)
At the start: 68.2 x 57 mm, 31 parts

Commit message: Optimized v9
Routing:
- net N$16: track 15.1 -> 14.3 mm, vias 2 -> 0
Changed lines of the file:
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@@
 <contactref element="R9" pad="2"/>
 <contactref element="U$4" pad="3"/>
-<wire x1="46.99" y1="20.32" x2="48.26" y2="21.59" width="0.254" layer="1"/>
-<wire x1="43.18" y1="20.32" x2="46.99" y2="20.32" width="0.254" layer="1"/>
-<wire x1="43.18" y1="22.86" x2="43.18" y2="20.32" width="0.254" layer="1"/>
-<wire x1="40.64" y1="25.4" x2="43.18" y2="22.86" width="0.254" layer="16"/>
-<wire x1="40.64" y1="22.86" x2="40.64" y2="25.4" width="0.254" layer="1"/>
 <wire x1="48.26" y1="21.59" x2="48.0147" y2="21.9681" width="0.254" layer="1"/>
 <wire x1="40.2691" y1="22.874" x2="40.64" y2="22.86" width="0.254" layer="1"/>
-<via x="43.18" y="22.86" extent="1-16" drill="0.6096"/>
-<via x="40.64" y="25.4" extent="1-16" drill="0.6096"/>
+<wire x1="40.64" y1="22.86" x2="40.3672" y2="22.86" width="0.254" layer="1"/>
+<wire x1="40.3672" y1="22.86" x2="40.3672" y2="19.6169" width="0.254" layer="1"/>
+<wire x1="40.3672" y1="19.6169" x2="48.0147" y2="19.6169" width="0.254" layer="1"/>
+<wire x1="48.0147" y1="19.6169" x2="48.0147" y2="21.9681" width="0.254" layer="1"/>
 </signal>
 <signal name="N$14">
@@
 <contactref element="U$4" pad="6"/>
 <wire x1="52.07" y1="20.32" x2="52.07" y2="21.59" width="0.254" layer="1"/>
-<wire x1="41.91" y1="20.32" x2="52.07" y2="20.32" width="0.254" layer="16"/>
-<wire x1="41.91" y1="20.32" x2="41.91" y2="35.56" width="0.254" layer="1"/>
+<wire x1="41.91" y1="20.6416" x2="52.07" y2="20.32" width="0.254" layer="16"/>
+<wire x1="41.91" y1="20.6416" x2="41.91" y2="35.56" width="0.254" layer="1"/>
 <wire x1="41.91" y1="35.56" x2="38.1" y2="39.37" width="0.254" layer="1"/>
 <wire x1="38.1" y1="39.37" x2="38.1" y2="48.26" width="0.254" layer="1"/>
@@
 <wire x1="27.4547" y1="56.2739" x2="27.94" y2="57.15" width="0.254" layer="1"/>
 <via x="52.07" y="20.32" extent="1-16" drill="0.6096"/>
-<via x="41.91" y="20.32" extent="1-16" drill="0.6096"/>
+<via x="41.91" y="20.6416" extent="1-16" drill="0.6096"/>
 <via x="38.1" y="48.26" extent="1-16" drill="0.6096"/>
 <via x="31.75" y="52.07" extent="1-16" drill="0.6096"/>
@@
 </signal>
 </signals>
-<errors>
-</errors>
 </board>
 </drawing>
